File: output/pcbs/quacken_pcb.kicad_pcb (KiCad board)
At the start: 2 copper layers, 262.2 x 120.5 mm, 87 parts

Commit message: Put capacitors on bottom side + better hotswap.
Parts:
- removed ? (x42): , Diode_SMD:D_SOD-323
- added D1: , Diode_SMD:D_SOD-323, B.Cu at (102.9, 121.3)
- added D10: , Diode_SMD:D_SOD-323, B.Cu at (157.5, 128.0)
- added D11: , Diode_SMD:D_SOD-323, B.Cu at (163.3, 112.0)
- added D12: , Diode_SMD:D_SOD-323, B.Cu at (169.1, 96.0)
- added D13: , Diode_SMD:D_SOD-323, B.Cu at (149.3, 150.3)
- added D14: , Diode_SMD:D_SOD-323, B.Cu at (168.8, 161.1)
- added D15: , Diode_SMD:D_SOD-323, B.Cu at (184.8, 176.6)
- added D16: , Diode_SMD:D_SOD-323, B.Cu at (303.1, 120.2)
- added D17: , Diode_SMD:D_SOD-323, B.Cu at (300.2, 103.5)
- added D18: , Diode_SMD:D_SOD-323, B.Cu at (297.2, 86.7)
- added D19: , Diode_SMD:D_SOD-323, B.Cu at (282.7, 114.1)
- added D2: , Diode_SMD:D_SOD-323, B.Cu at (105.9, 104.6)
- added D20: , Diode_SMD:D_SOD-323, B.Cu at (278.0, 97.8)
- added D21: , Diode_SMD:D_SOD-323, B.Cu at (273.4, 81.5)
- added D22: , Diode_SMD:D_SOD-323, B.Cu at (263.7, 115.6)
- added D23: , Diode_SMD:D_SOD-323, B.Cu at (257.9, 99.6)
- added D24: , Diode_SMD:D_SOD-323, B.Cu at (252.1, 83.7)
- added D25: , Diode_SMD:D_SOD-323, B.Cu at (248.3, 125.8)
- added D26: , Diode_SMD:D_SOD-323, B.Cu at (242.4, 109.8)
- added D27: , Diode_SMD:D_SOD-323, B.Cu at (236.6, 93.8)
- added D28: , Diode_SMD:D_SOD-323, B.Cu at (256.4, 148.1)
- added D29: , Diode_SMD:D_SOD-323, B.Cu at (236.2, 157.5)
- added D3: , Diode_SMD:D_SOD-323, B.Cu at (108.8, 87.9)
- added D30: , Diode_SMD:D_SOD-323, B.Cu at (219.1, 171.7)
- added D31: , Diode_SMD:D_SOD-323, B.Cu at (77.8, 123.4)
- added D32: , Diode_SMD:D_SOD-323, B.Cu at (80.7, 106.7)
- added D33: , Diode_SMD:D_SOD-323, B.Cu at (83.7, 89.9)
- added D34: , Diode_SMD:D_SOD-323, B.Cu at (166.2, 137.9)
- added D35: , Diode_SMD:D_SOD-323, B.Cu at (172.0, 121.9)
- added D36: , Diode_SMD:D_SOD-323, B.Cu at (177.9, 105.9)
- added D37: , Diode_SMD:D_SOD-323, B.Cu at (315.7, 124.5)
- added D38: , Diode_SMD:D_SOD-323, B.Cu at (312.7, 107.8)
- added D39: , Diode_SMD:D_SOD-323, B.Cu at (309.7, 91.0)
- added D4: , Diode_SMD:D_SOD-323, B.Cu at (123.2, 115.9)
- added D40: , Diode_SMD:D_SOD-323, B.Cu at (227.5, 140.0)
- added D41: , Diode_SMD:D_SOD-323, B.Cu at (221.7, 124.1)
- added D42: , Diode_SMD:D_SOD-323, B.Cu at (215.9, 108.1)
- added D5: , Diode_SMD:D_SOD-323, B.Cu at (127.8, 99.6)
- added D6: , Diode_SMD:D_SOD-323, B.Cu at (132.5, 83.2)
- added D7: , Diode_SMD:D_SOD-323, B.Cu at (142.0, 117.8)
- added D8: , Diode_SMD:D_SOD-323, B.Cu at (147.8, 101.8)
- added D9: , Diode_SMD:D_SOD-323, B.Cu at (153.7, 85.9)
- moved S39 227.8 mm to (312.6, 89.0), turned to 10 degrees
- moved S28 159.2 mm to (253.9, 150.6), turned to -160 degrees
- moved S35 141.4 mm to (175.6, 121.6), turned to -20 degrees
- moved S14 135.9 mm to (165.3, 160.5), turned to 145 degrees
- moved S27 135.1 mm to (234.1, 96.3), turned to -160 degrees
- moved S36 132.6 mm to (181.4, 105.6), turned to -20 degrees
- moved S15 108.0 mm to (181.6, 175.1), turned to 130 degrees
- moved S30 106.4 mm to (218.2, 175.1), turned to -130 degrees
- moved S33 99.6 mm to (87.1, 89.0), turned to -10 degrees
- moved S38 96.9 mm to (315.6, 105.7), turned to 10 degrees
- moved S37 94.0 mm to (318.5, 122.5), turned to 10 degrees
- moved S41 89.3 mm to (224.2, 121.6), turned to 20 degrees
- moved S26 76.6 mm to (240.0, 112.3), turned to -160 degrees
- moved S29 75.7 mm to (234.4, 160.5), turned to -145 degrees
- moved S24 74.4 mm to (249.6, 86.2)
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Connections:
- S1 pad 1: P16 -> pinky_bottom
- S1 pad 2: pinky_bottom -> P14
- S10 pad 1: P8 -> index_bottom
- S10 pad 2: index_top -> P7
- S11 pad 1: P7 -> index_home
- S11 pad 2: tucky_default -> P7
- S12 pad 1: P8 -> index_top
- S12 pad 2: comfy_default -> P7
- S13 pad 1: P9 -> tucky_default
- S13 pad 2: reachy_default -> P8
- S14 pad 1: P16 -> comfy_default
- S14 pad 2: mirror_pinky_bottom -> P7
- S15 pad 1: P14 -> reachy_default
- S15 pad 2: mirror_ring_bottom -> P6
- S16 pad 1: P14 -> mirror_pinky_bottom
- S16 pad 2: mirror_ring_home -> P14
- S17 pad 1: P14 -> mirror_pinky_home
- S17 pad 2: mirror_ring_top -> P14
- S18 pad 1: P7 -> mirror_pinky_top
- S18 pad 2: mirror_middle_bottom -> P14
- S19 pad 1: P7 -> mirror_ring_bottom
- S19 pad 2: mirror_middle_home -> P15
- S2 pad 1: P14 -> pinky_home
- S2 pad 2: ring_bottom -> P14
- S20 pad 1: P7 -> mirror_ring_home
- S20 pad 2: mirror_middle_top -> P15
- S21 pad 1: P8 -> mirror_ring_top
- S21 pad 2: mirror_index_bottom -> P15
- S22 pad 1: P8 -> mirror_middle_bottom
- S22 pad 2: mirror_index_home -> P8
- S23 pad 1: P8 -> mirror_middle_home
- S23 pad 2: mirror_index_top -> P8
- S24 pad 1: P7 -> mirror_middle_top
- S24 pad 2: mirror_tucky_default -> P8
- S25 pad 1: P8 -> mirror_index_bottom
- S25 pad 2: mirror_comfy_default -> P7
- S26 pad 1: P9 -> mirror_index_home
- S26 pad 2: mirror_reachy_default -> P7
- S27 pad 1: P16 -> mirror_index_top
- S27 pad 2: pinky_home -> P7
- S28 pad 1: P16 -> mirror_tucky_default
- S28 pad 2: pinky_top -> P8
- S29 pad 1: P16 -> mirror_comfy_default
- S29 pad 2: mirror_pinky_home -> P7
- S3 pad 1: P14 -> pinky_top
- S3 pad 2: ring_home -> P14
- S30 pad 1: P16 -> mirror_reachy_default
- S30 pad 2: mirror_pinky_top -> P6
- S31 pad 1: P10 -> outer_bottom
- S31 pad 2: outer_bottom -> P16
- S31 pad 3: P10 -> P16
- S32 pad 1: P10 -> outer_home
- S32 pad 2: outer_home -> P16
- S32 pad 3: P10 -> P16
- S33 pad 1: P9 -> outer_top
- S33 pad 2: inner_bottom -> P16
- S34 pad 1: P9 -> inner_bottom
- S34 pad 2: inner_home -> P6
- S34 pad 3: P9 -> P6
- S35 pad 1: P10 -> inner_home
- S35 pad 2: mirror_outer_bottom -> P6
- S35 pad 3: P10 -> P6
- S36 pad 1: P10 -> inner_top
- S36 pad 2: mirror_outer_home -> P6
- S37 pad 1: P9 -> mirror_outer_bottom
- S37 pad 2: mirror_inner_bottom -> P16
- S37 pad 3: P9 -> P16
- S38 pad 1: P9 -> mirror_outer_home
- S38 pad 2: mirror_inner_home -> P16
- S38 pad 3: P9 -> P16
- S39 pad 1: P10 -> mirror_outer_top
- S39 pad 2: outer_top -> P16
- S4 pad 1: P14 -> ring_bottom
- S4 pad 2: ring_top -> P15
- S40 pad 1: P9 -> mirror_inner_bottom
- S40 pad 2: inner_top -> P6
- S41 pad 1: P10 -> mirror_inner_home
- S41 pad 2: mirror_outer_top -> P6
- S42 pad 1: P9 -> mirror_inner_top
- S42 pad 2: mirror_inner_top -> P6
- S5 pad 1: P7 -> ring_home
- S5 pad 2: middle_bottom -> P15
- S6 pad 1: P7 -> ring_top
- S6 pad 2: middle_home -> P15
- S7 pad 1: P7 -> middle_bottom
- S7 pad 2: middle_top -> P8
- S8 pad 1: P8 -> middle_home
- S8 pad 2: index_bottom -> P8
- S9 pad 1: P8 -> middle_top
- S9 pad 2: index_home -> P8
Routing:
- net P10: track 372.4 -> 72.4 mm, vias 2 -> 3
- net P6: track 85.1 -> 291.4 mm
- net P9: track 255.7 -> 75.4 mm, vias 0 -> 5
- net P15: track 77.7 -> 255.2 mm
- net P7: track 345.6 -> 248.1 mm
- net P16: track 329.9 -> 394.7 mm
- net P14: track 296.7 -> 332.8 mm
- net P19: track 120.1 -> 139.1 mm, vias 0 -> 6
- net GND: track 18.4 -> 0.00 mm, vias 0 -> 23
- net P20: track 130.7 -> 148.9 mm, vias 0 -> 6
- net mirror_inner_top: track 22.0 -> 6.20 mm, vias 1 -> 0
- net mirror_outer_top: track 21.8 -> 6.20 mm, vias 1 -> 0
- net P3: track 132.3 -> 147.4 mm, vias 0 -> 6
- net pinky_bottom: track 20.8 -> 6.20 mm, vias 1 -> 0
- net P4: track 123.1 -> 134.9 mm, vias 0 -> 6
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- added copper zone on B.Cu, net GND
- added copper zone on F.Cu, net GND
Other:
- outline, holes or cut-outs redrawn
- board text removed: "Quacken v0"
